File: ai03_pcb_guide.kicad_pcb (KiCad board)
At the start: 2 copper layers, 79.4 x 38.1 mm, 24 parts, among them SW1 SW_Push, U1 ATmega32U4-A, Y1 16 MHz

Commit message: routing
Parts:
- moved C2 5.07 mm to (63.6, 68.4)
- moved Y1 4.79 mm to (67.8, 68.5)
- moved C1 4.79 mm to (71.9, 68.5)
- moved C3 1.66 mm to (54.0, 79.0)
Connections:
- U1 pad 27: unconnected-(U1-Pad27) -> /ROW0
- U1 pad 28: unconnected-(U1-Pad28) -> /COL1
- U1 pad 29: unconnected-(U1-Pad29) -> /COL0
- U1 pad 30: unconnected-(U1-Pad30) -> /ROW1
Routing:
- net GND: track 0.00 -> 134.5 mm
- net +5V: track 0.00 -> 98.0 mm, vias 0 -> 5
- net /ROW1: track 0.00 -> 56.4 mm
- net /COL1: track 0.00 -> 55.9 mm
- net /ROW0: track 0.00 -> 51.7 mm
- net /COL0: track 0.00 -> 37.4 mm
- net Net-(R3-Pad2): track 0.00 -> 20.9 mm
- net Net-(R2-Pad2): track 0.00 -> 20.2 mm
- net Net-(R1-Pad2): track 0.00 -> 20.1 mm, vias 0 -> 2
- net Net-(C2-Pad2): track 0.00 -> 12.2 mm
- net Net-(C1-Pad2): track 0.00 -> 11.6 mm
- net VCC: track 0.00 -> 10.2 mm
- net Net-(D4-Pad2): track 0.00 -> 7.41 mm
- net Net-(D3-Pad2): track 0.00 -> 6.82 mm
- net Net-(D2-Pad2): track 0.00 -> 6.82 mm
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
Commit message: end of guide edits
Routing:
- net Net-(R1-Pad2): track 20.1 -> 29.0 mm
- net +5V: track 98.0 -> 103.8 mm, vias 5 -> 6
- added copper zone on B.Cu, net GND
Other:
- board text added: "BRIDGET'S PCB"
